File: Board/stm32ext.brd (EAGLE design)
At the start: 0 parts

Commit message: Board finalized. COM receive needs some work.
Routing:
- net S$19: track 53.1 -> 5.26 mm
- net S$129: track 0.00 -> 46.6 mm, vias 1 -> 0
- net S$37: track 0.00 -> 42.8 mm
- net S$126: track 50.2 -> 8.89 mm
- net S$18: track 44.6 -> 5.26 mm
- net S$72: track 0.00 -> 37.9 mm
- net S$119: track 0.00 -> 35.5 mm
- net S$151: track 0.00 -> 34.1 mm
- net S$50: track 0.00 -> 27.9 mm
- net S$4: track 0.00 -> 27.5 mm, vias 0 -> 1
- net S$7: track 82.2 -> 55.2 mm, vias 1 -> 0
- net S$2: track 0.00 -> 27.0 mm
- net S$122: track 61.2 -> 34.3 mm
- net S$121: track 26.6 -> 0.00 mm
- net S$131: track 0.00 -> 22.0 mm
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- added copper zone on layer 1, net GND
- added copper zone on layer 16, net GND
Other:
- board outline added: 91.4 x 97.8 mm
- board text added: "GPIO0(PE6)"
- board text added: "GPIO1(PE7)"
- board text added: "PA0"
- board text added: "PE6"
- board text added: "PE7"
- board text added: "UART4_RX"
- board text added: "UART4_TX"
- board text removed: "50Ω"
- board text removed: "IN10"
- board text removed: "IN3"
- board text removed: "IN4"
- board text removed: "IN5"
- board text removed: "IN6"
- board text removed: "IN7"
- board text removed: "IN8"
- board text removed: "IN9"
- board text removed: "PA10"
- board text removed: "PA4"
- board text removed: "PA5"
- board text removed: "PA6"
- board text removed: "PA7"
- board text removed: "PA8"
- board text removed: "PA9"
- board text removed: "PB13"
